Commit message: Fix double pendulum URDF model and configuration `configRobot.m`
- mode.urdf: fix robot name, add high mass and inertia to the world link,
  replace continuous by revolute joints, replace dae mesh by box shape.
- configRobot.m: list of controlled joints, mesh file prefix, initial conditions,
  Frames (BASE is the 'world' link, which is heavy enough to be considered fixed,
  and that base frame is also used as LEFT_FOOT/RIGHT_FOOT)
  For emulating a fixed base, the contact vertices are set far away from the frame
  origin, and the friction coefficient set to very high value.

File: urdf/RRbot/robots/RRbot1/model.urdf (robot description, URDF)
Before this commit: robot single_rrbot, 6 links, 5 joints
Links:
- removed link single_rrbot_camera_link
- removed link single_rrbot_hokuyo_link
- removed link single_rrbot_link1
- removed link single_rrbot_link2
- removed link single_rrbot_link3
- added link RRbot_camera_link, mass 1e-5; collision box size=0.05 0.05 0.05; visual box size=0.05 0.05 0.05
- added link RRbot_hokuyo_link, mass 1e-5; collision box size=0.1 0.1 0.1; visual box size=0.1 0.1 0.1
- added link RRbot_link1, mass 1; collision box size=0.1 0.1 2; visual box size=0.1 0.1 2
- added link RRbot_link2, mass 1; collision box size=0.1 0.1 1; visual box size=0.1 0.1 1
- added link RRbot_link3, mass 1; collision box size=0.1 0.1 1; visual box size=0.1 0.1 1
- link world: mass None -> 1000
Joints:
- removed joint single_rrbot_camera_joint
- removed joint single_rrbot_fixed
- removed joint single_rrbot_hokuyo_joint
- removed joint single_rrbot_joint1
- removed joint single_rrbot_joint2
- added joint RRbot_camera_joint: type fixed, parent RRbot_link3, child RRbot_camera_link, origin xyz=0.05 0 0.9 rpy=0 0 0, axis 0 1 0
- added joint RRbot_fixed: type fixed, parent world, child RRbot_link1, origin xyz=0 0 0 rpy=0 0 0
- added joint RRbot_hokuyo_joint: type fixed, parent RRbot_link3, child RRbot_hokuyo_link, origin xyz=0 0 0.975 rpy=0 0 0, axis 0 1 0
- added joint RRbot_joint1: type revolute, parent RRbot_link1, child RRbot_link2, origin xyz=0 0.1 1.95 rpy=0 0 0, axis 0 1 0
- added joint RRbot_joint2: type revolute, parent RRbot_link2, child RRbot_link3, origin xyz=0 0.1 0.9 rpy=0 0 0, axis 0 1 0

Commit message: Fixed #23: converted RRbot1 mesh from DAE to STL and added to model

File: urdf/RRbot/robots/RRbot1/model.urdf (robot description, URDF)
Before this commit: robot RRbot, 6 links, 5 joints
Links:
- link RRbot_hokuyo_link: geometry collision box size=0.1 0.1 0.1; visual mesh filename=package://RRbot/meshes/hokuyo.stl
